Commit message: Updated rover xacro and created lidar xacro

File: urdf/rover.urdf.xacro (robot description, xacro)
@@ -9,5 +9,5 @@
   <xacro:property name="leg_width" value="0.02" />
   <xacro:property name="leg_length" value="0.02" />
-  <gazebo reference="body">
+ <gazebo reference="body">
     <material>Gazebo/White</material>
     <mu1>0.2</mu1>
@@ -129,4 +129,10 @@
     <dynamics friction="0.5"/>
   </joint>
+  <xacro:include filename="$(find robot_tutorial_3)/urdf/lidar.urdf.xacro"/>
+  <joint name="lidarGlue" type="fixed">
+    <parent link="body"/>
+    <child link="laz_base"/>
+    <origin xyz="0 0 ${body_height/2}"/>
+  </joint>
   <gazebo>
     <plugin name="rover_plugin" filename="librover_plugin.so"> </plugin>
